File: lora1276Breakout.kicad_pcb (KiCad board)
At the start: 2 copper layers, 39.4 x 27.9 mm, 9 parts, among them J1 Conn_01x10_Male, U1 Lora1276_V2.0

Commit message: update to latest kicad and small changes
Parts:
- renumbered SMA to J2, u.FL to J3
Connections:
- net Net-(J1-Pad1) renamed /SCK
- net Net-(J1-Pad2) renamed /MISO
- net Net-(J1-Pad3) renamed /MOSI
- net Net-(J1-Pad4) renamed /CS
- net Net-(J1-Pad5) renamed /DIO2
- net Net-(J1-Pad6) renamed /DIO1
- net Net-(J1-Pad7) renamed /DIO0
- net Net-(J1-Pad8) renamed /RESET
- U1 pad 2: (no net) -> unconnected-(U1-Pad2)
- U1 pad 3: (no net) -> unconnected-(U1-Pad3)
Other:
- net class Default removed
